File: hardware/kicad/ionos_maximus.kicad_pcb (KiCad board)
At the start: 2 copper layers, 45 x 39.1 mm, 45 parts, among them J1 CLH-115-F-D-DV, J2 NA(TC2030-NL), P200 TFC-120-02-F-D-A-K-TR, P201 TFC-120-02-F-D-A-K-TR, U1 LP5907MFX-3.3, U2 CAT24C32WI-GT3

Commit message: P200 board-ID I2C as on ionos-sdr-mini: JP9/JP10 cut points, R18/R19 4.7k pull-ups (DNP, the Pi has 1k8)
Parts:
- added JP10: Bridged, Jumper:SolderJumper-2_P1.3mm_Bridged_RoundedPad1.0x1.5mm, F.Cu at (10.6, -1.90)
- added JP9: Bridged, Jumper:SolderJumper-2_P1.3mm_Bridged_RoundedPad1.0x1.5mm, F.Cu at (10.6, -4.60)
- added R18: NA(4.7k), ionos_maximus:RESC1005X40_0402, F.Cu at (13.0, -5.20)
- added R19: NA(4.7k), ionos_maximus:RESC1005X40_0402, F.Cu at (13.0, -2.20)
Connections:
- P200 pad 39: I2C_SCL -> I2C_SCL_RB
- P200 pad 40: I2C_SDA -> I2C_SDA_RB
