File: hardware/kicad/ionos_maximus.kicad_sch (KiCad schematic)
At the start: 49 parts, among them J1 CLH-115-F-D-DV, J2 NA(TC2030-NL), P200 TFC-120-02-F-D-A-K-TR, P201 TFC-120-02-F-D-A-K-TR, U1 LP5907MFX-3.3, U2 CAT24C32WI-GT3

Commit message: hardware: rev A routed, realistic 3D renders
- Board routed on 2 layers with GND pour on both sides.
  DRC: 0 errors, 0 unconnected, schematic parity 0.
- J2 (TC2030, DNP) removed. U2 changed to TSSOP-8 and moved to
  the P200/P201 band.
- 3V3_PI taken from RPi pin 17 only. Rule-area keepout over the slot.
- gen/render_context.py: Pi 3 + radio board + SMA antenna context
  renders, built from KiCad library stand-ins.
- README images updated.

Co-Authored-By: Claude Opus 5.5 <noreply@anthropic.com>
Claude-Session: https://claude.ai/code/session_01NdGLVAcWNnBXKQpCaswFNe
Parts:
- removed J2: NA(TC2030-NL), Connector:Tag-Connect_TC2030-IDC-NL_2x03_P1.27mm_Vertical, symbol ionos_maximus:TC2030
- U2: value CAT24C32WI-GT3 -> CAT24C32YI-GT3; footprint Package_SO:SOIC-8_3.9x4.9mm_P1.27mm -> Package_SO:TSSOP-8_4.4x3mm_P0.65mm
Connections:
- net 3V3_PI: no longer J1.2 (3V3 [1])
- net IQ_CS: now reaches R5.2, R6.1, R7.1
- net IQ_CS_PI: now reaches JP3.2 (B), R5.1
- net IQ_SCLK_PI: now reaches JP2.2 (B), R3.1
- net IQ_SCLK: now reaches R3.2, R4.1
- net DRDY: now reaches R10.2, R11.1, R12.1, TP1.PP
- net VRF_IN: now reaches P201.40, TP6.PP
- net IQ_DATA: now reaches R8.2, R9.1
- no-connect marks 67 -> 68
Other:
- note added: "Cut JP4-JP7 to drive SWD from an external probe (radio-board side"
- note added: "Pi 3V3 (pin 17 only) feeds only the ID EEPROM. ID_SD / ID_SC: EEPROM + 3.9k only."
- note added: "of the cut points). RESETn: open-drain only."
- note removed: "(Tag-Connect TC2030-NL, not fitted). RESETn: open-drain only."
- note removed: "Cut JP4-JP7 to use an external probe on J2"
- note removed: "Pi 3V3 (1, 17) feeds only the ID EEPROM. ID_SD / ID_SC: EEPROM + 3.9k only."
- moved on the sheet: R10, R11, R12, R13, R14, R3, R4, R5, R6, R7, R8, R9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
